Commit message: Update the xacro based on the test on real j2n6s300 robot

File: kinova_description/urdf/j2n6s300.xacro (robot description, xacro)
@@ -80,10 +80,10 @@
     <xacro:property name="joint_4_torque_limit" value="20" />
     <xacro:property name="joint_5" value="joint_5" />
-    <xacro:property name="joint_5_type" value="continuous" />
+    <xacro:property name="joint_5_type" value="revolute" />
     <xacro:property name="joint_5_axis_xyz" value="0 0 1" />
     <xacro:property name="joint_5_origin_xyz" value="0 -0.03703 -0.06414" />
     <xacro:property name="joint_5_origin_rpy" value="${J_PI/3} 0 ${J_PI}" />
-    <xacro:property name="joint_5_lower_limit" value="${-2*J_PI}" />
-    <xacro:property name="joint_5_upper_limit" value="${2*J_PI}" />
+    <xacro:property name="joint_5_lower_limit" value="${66/180*J_PI}" />
+    <xacro:property name="joint_5_upper_limit" value="${294/180*J_PI}" />
     <xacro:property name="joint_5_velocity_limit" value="${48*J_PI/180}" />
     <xacro:property name="joint_5_torque_limit" value="20" />

Commit message: Update joint_5_type to continuous and adjust joint_5 limits in j2n6s300.xacro (problem fixed by updating jaco firmware)

File: kinova_description/urdf/j2n6s300.xacro (robot description, xacro)
@@ -80,10 +80,10 @@
     <xacro:property name="joint_4_torque_limit" value="20" />
     <xacro:property name="joint_5" value="joint_5" />
-    <xacro:property name="joint_5_type" value="revolute" />
+    <xacro:property name="joint_5_type" value="continuous" />
     <xacro:property name="joint_5_axis_xyz" value="0 0 1" />
     <xacro:property name="joint_5_origin_xyz" value="0 -0.03703 -0.06414" />
     <xacro:property name="joint_5_origin_rpy" value="${J_PI/3} 0 ${J_PI}" />
-    <xacro:property name="joint_5_lower_limit" value="${66/180*J_PI}" />
-    <xacro:property name="joint_5_upper_limit" value="${294/180*J_PI}" />
+    <xacro:property name="joint_5_lower_limit" value="${-2*J_PI}" />
+    <xacro:property name="joint_5_upper_limit" value="${2*J_PI}" />
     <xacro:property name="joint_5_velocity_limit" value="${48*J_PI/180}" />
     <xacro:property name="joint_5_torque_limit" value="20" />

Commit message: refactor: Update joint_end_effector_origin_xyz  in j2n6s300.xacro -> move ee frame inward for grasping

File: kinova_description/urdf/j2n6s300.xacro (robot description, xacro)
@@ -102,5 +102,6 @@
     <xacro:property name="joint_end_effector_type" value="fixed" />
     <xacro:property name="joint_end_effector_axis_xyz" value="0 0 0" />
-    <xacro:property name="joint_end_effector_origin_xyz" value="0 0 -0.1600" />
+    <!-- <xacro:property name="joint_end_effector_origin_xyz" value="0 0 -0.1600" /> -->
+    <xacro:property name="joint_end_effector_origin_xyz" value="0 0 -0.1200" />
     <xacro:property name="joint_end_effector_origin_rpy" value="${J_PI} 0 ${J_PI/2}" />
     <xacro:macro name="j2n6s300" params="base_parent prefix:=j2n6s300">
